Commit message: table joints

File: robots_ee_pkg/urdf/kuka_robot/kuka_iiwa7.gazebo.xacro (robot description, xacro)
@@ -60,11 +60,4 @@
       <mu2>0.2</mu2>
     </gazebo>
-    <gazebo reference="${robot_name}_table_base_primary">
-      <material>Gazebo/Black</material>
-      <turnGravityOff>true</turnGravityOff>
-      <legacyModeNS>true</legacyModeNS>
-      <mu1>0.1</mu1>
-      <mu2>0.1</mu2>
-    </gazebo>
     <gazebo>
       <plugin name="gazebo_ros_control" filename="libgazebo_ros_control.so">
