Commit message: Table plugin

File: robots_ee_pkg/urdf/table/add_table.urdf.xacro (robot description, xacro)
@@ -9,7 +9,9 @@
       <xacro:insert_block name="origin"/>
       <parent link="${parent}"/>
-      <child link="${robot_arm_name}_table_fixed_link"/>
+      <!--child link="${robot_arm_name}_table_fixed_link"/ -->
+      <!--child link="${robot_arm_name}_table_yaw_link"/-->
+      <child link="${robot_arm_name}_table_base"/>
     </joint>
-    <joint name="${robot_arm_name}_table_x_joint" type="prismatic">
+    <!--joint name="${robot_arm_name}_table_x_joint" type="prismatic">
       <origin xyz="0 0 0" rpy="0 0 0"/>
       <parent link="${robot_arm_name}_table_fixed_link"/>
@@ -23,7 +25,7 @@
       <child link="${robot_arm_name}_table_yaw_link"/>
       <axis xyz="0 0 1" />
-    </joint>
+    </joint-->
     <!-- Extra links-->
-    <link name="${robot_arm_name}_table_fixed_link">
+    <!--link name="${robot_arm_name}_table_fixed_link">
       <inertial>
         <mass value="1"/>
@@ -56,7 +58,7 @@
         </material>
       </visual>
-    </link>
+    </link-->
      <!-- BASE LINK -->
-    <link name="${robot_arm_name}_table_yaw_link">
+    <link name="${robot_arm_name}_table_base">
       <inertial>
         <mass value="80"/>
@@ -81,5 +83,5 @@
       </collision>
     </link>
-    <gazebo reference="${robot_arm_name}_table_yaw_link">
+    <gazebo reference="${robot_arm_name}_table_base">
       <material>Gazebo/Grey</material>
       <turnGravityOff>true</turnGravityOff>
@@ -89,5 +91,5 @@
     <joint name="${robot_arm_name}_table_base_top_joint" type="fixed">
       <origin rpy="0 0 0" xyz="0.0 0 0.015"/>
-      <parent link="${robot_arm_name}_table_yaw_link"/>
+      <parent link="${robot_arm_name}_table_base"/>
       <child link="${table_ee}"/>
     </joint>
@@ -122,5 +124,5 @@
       <mu2>0.4</mu2>
     </gazebo>
-    <gazebo reference="${robot_arm_name}_table_fixed_link">
+    <!--gazebo reference="${robot_arm_name}_table_fixed_link">
       <material>Gazebo/Grey</material>
       <selfCollide>false</selfCollide>
@@ -155,5 +157,5 @@
             <mechanicalReduction>1</mechanicalReduction>
         </actuator>
-    </transmission>
+    </transmission -->
   </xacro:macro>
 </robot>
