Commit message: new workplace

File: robots_ee_pkg/urdf/conveyor/conveyor.urdf.xacro (robot description, xacro)
@@ -32,6 +32,6 @@
     </link>
     <gazebo reference="conveyor_system_link">
-      <material>Gazebo/Silver</material>
-      <turnGravityOff>false</turnGravityOff>
+      <material>Gazebo/Black</material>
+      <gravity>true</gravity>
       <mu1>0.5</mu1>
       <mu2>0.4</mu2>
