Commit message: panda update

File: robots_ee_pkg/urdf/panda_robot/panda.gazebo.xacro (robot description, xacro)
@@ -11,5 +11,5 @@
     <!-- Link0 -->
     <gazebo reference="${arm_name}_link0">
-      <material>Gazebo/Grey</material>
+      <material>Gazebo/White</material>
       <mu1>0.61</mu1>
       <mu2>0.61</mu2>
@@ -17,5 +17,5 @@
     <!-- Link1 -->
     <gazebo reference="${arm_name}_link1">
-      <material>Gazebo/Grey</material>
+      <material>Gazebo/White</material>
       <mu1>0.2</mu1>
       <mu2>0.2</mu2>
@@ -23,5 +23,5 @@
     <!-- Link2 -->
     <gazebo reference="${arm_name}_link2">
-      <material>Gazebo/Grey</material>
+      <material>Gazebo/White</material>
       <mu1>0.2</mu1>
       <mu2>0.2</mu2>
@@ -29,5 +29,5 @@
     <!-- Link3 -->
     <gazebo reference="${arm_name}_link3">
-      <material>Gazebo/Grey</material>
+      <material>Gazebo/White</material>
       <mu1>0.2</mu1>
       <mu2>0.2</mu2>
@@ -35,5 +35,5 @@
     <!-- Link4 -->
     <gazebo reference="${arm_name}_link4">
-      <material>Gazebo/Grey</material>
+      <material>Gazebo/White</material>
       <mu1>0.2</mu1>
       <mu2>0.2</mu2>
@@ -41,5 +41,5 @@
     <!-- Link5 -->
     <gazebo reference="${arm_name}_link5">
-      <material>Gazebo/Grey</material>
+      <material>Gazebo/White</material>
       <mu1>0.2</mu1>
       <mu2>0.2</mu2>
@@ -47,5 +47,5 @@
     <!-- Link6 -->
     <gazebo reference="${arm_name}_link6">
-      <material>Gazebo/Grey</material>>
+      <material>Gazebo/White</material>>
       <mu1>0.2</mu1>
       <mu2>0.2</mu2>
@@ -53,5 +53,5 @@
     <!-- Link7 -->
     <gazebo reference="${arm_name}_link7">
-      <material>Gazebo/Grey</material>
+      <material>Gazebo/White</material>
       <mu1>0.2</mu1>
       <mu2>0.2</mu2>
