Commit message: panda update

File: franka_ros-kinetic-devel/franka_description/robots/hand.xacro (robot description, xacro)
@@ -20,4 +20,9 @@
         </geometry>
       </collision>
+      <inertial>
+        <origin xyz="0 0 0" rpy="0 0 0" />
+        <mass value="0.67893">
+        <inertia ixx="0.3" ixy="0.0" ixz="0.0" iyy="0.3" iyz="0.0" izz="0.3" />
+      </inertial>
     </link>
     <link name="${ns}_leftfinger">
@@ -32,4 +37,9 @@
         </geometry>
       </collision>
+      <inertial>
+        <origin xyz="0 0 0" rpy="0 0 0" />
+        <mass value="0.01053">
+        <inertia ixx="0.3" ixy="0.0" ixz="0.0" iyy="0.3" iyz="0.0" izz="0.3" />
+      </inertial>
     </link>
     <link name="${ns}_rightfinger">
@@ -46,4 +56,9 @@
         </geometry>
       </collision>
+      <inertial>
+        <origin xyz="0 0 0" rpy="0 0 0" />
+        <mass value="0.01053">
+        <inertia ixx="0.3" ixy="0.0" ixz="0.0" iyy="0.3" iyz="0.0" izz="0.3" />
+      </inertial>
     </link>
     <joint name="${ns}_finger_joint1" type="prismatic">

File: franka_ros-kinetic-devel/franka_description/robots/panda_arm.xacro (robot description, xacro)
@@ -1,4 +1,5 @@
 <?xml version='1.0' encoding='utf-8'?>
 <robot xmlns:xacro="http://www.ros.org/wiki/xacro" name="panda">
+  <xacro:property name="joint_damping" value = "1.0" />
   <xacro:macro name="panda_arm" params="arm_id:='panda' description_pkg:='franka_description' connected_to:='' xyz:='0 0 0' rpy:='0 0 0'">
     <xacro:unless value="${not connected_to}">
@@ -7,4 +8,5 @@
         <child link="${arm_id}_link0"/>
         <origin rpy="${rpy}" xyz="${xyz}"/>
+        <dynamic damping="${joint_damping}">
       </joint>
     </xacro:unless>
@@ -20,4 +22,9 @@
         </geometry>
       </collision>
+      <inertial>
+        <origin xyz="0 0 0" rpy="0 0 0" />
+        <mass value="3.06357">
+        <inertia ixx="0.3" ixy="0.0" ixz="0.0" iyy="0.3" iyz="0.0" izz="0.3" />
+      </inertial>
     </link>
     <link name="${arm_id}_link1">
@@ -32,4 +39,9 @@
         </geometry>
       </collision>
+      <inertial>
+        <origin xyz="0 0 0" rpy="0 0 0" />
+        <mass value="2.34471">
+        <inertia ixx="0.3" ixy="0.0" ixz="0.0" iyy="0.3" iyz="0.0" izz="0.3" />
+      </inertial>
     </link>
     <joint name="${arm_id}_joint1" type="revolute">
@@ -52,4 +64,9 @@
         </geometry>
       </collision>
+      <inertial>
+        <origin xyz="0 0 0" rpy="0 0 0" />
+        <mass value="2.36414">
+        <inertia ixx="0.3" ixy="0.0" ixz="0.0" iyy="0.3" iyz="0.0" izz="0.3" />
+      </inertial>
     </link>
     <joint name="${arm_id}_joint2" type="revolute">
@@ -72,4 +89,9 @@
         </geometry>
       </collision>
+      <inertial>
+        <origin xyz="0 0 0" rpy="0 0 0" />
+        <mass value="2.38050">
+        <inertia ixx="0.3" ixy="0.0" ixz="0.0" iyy="0.3" iyz="0.0" izz="0.3" />
+      </inertial>
     </link>
     <joint name="${arm_id}_joint3" type="revolute">
@@ -92,4 +114,9 @@
         </geometry>
       </collision>
+      <inertial>
+        <origin xyz="0 0 0" rpy="0 0 0" />
+        <mass value="2.42754">
+        <inertia ixx="0.3" ixy="0.0" ixz="0.0" iyy="0.3" iyz="0.0" izz="0.3" />
+      </inertial>
     </link>
     <joint name="${arm_id}_joint4" type="revolute">
@@ -112,4 +139,9 @@
         </geometry>
       </collision>
+      <inertial>
+        <origin xyz="0 0 0" rpy="0 0 0" />
+        <mass value="3.49611">
+        <inertia ixx="0.3" ixy="0.0" ixz="0.0" iyy="0.3" iyz="0.0" izz="0.3" />
+      </inertial>
     </link>
     <joint name="${arm_id}_joint5" type="revolute">
@@ -132,4 +164,9 @@
         </geometry>
       </collision>
+      <inertial>
+        <origin xyz="0 0 0" rpy="0 0 0" />
+        <mass value="1.46736">
+        <inertia ixx="0.3" ixy="0.0" ixz="0.0" iyy="0.3" iyz="0.0" izz="0.3" />
+      </inertial>
     </link>
     <joint name="${arm_id}_joint6" type="revolute">
@@ -152,4 +189,9 @@
         </geometry>
       </collision>
+      <inertial>
+        <origin xyz="0 0 0" rpy="0 0 0" />
+        <mass value="0.45606">
+        <inertia ixx="0.3" ixy="0.0" ixz="0.0" iyy="0.3" iyz="0.0" izz="0.3" />
+      </inertial>
     </link>
     <joint name="${arm_id}_joint7" type="revolute">

File: robots_ee_pkg/urdf/iwt_environment.xacro (robot description, xacro)
@@ -25,8 +25,8 @@
   </xacro:kuka_iiwa7_table_urdf>
   <!-- Franka Panda-->
-  <!--xacro:include filename="$(find robots_ee_pkg)/urdf/panda_robot/franka_panda.urdf.xacro" />
+  <xacro:include filename="$(find robots_ee_pkg)/urdf/panda_robot/franka_panda.urdf.xacro" />
   <xacro:franka_panda_table_urdf table_prefix="panda" table_parent="world_interface">
-    <origin xyz="0.5 0 1.0" rpy="0 0 ${pi/2}" />
-  </xacro:franka_panda_table_urdf-->
+    <origin xyz="3.7 -0.5 1.0" rpy="0 0 ${pi/2}" />
+  </xacro:franka_panda_table_urdf>
   <!-- ur5-->
   <xacro:include filename="$(find robots_ee_pkg)/urdf/ur5_robot/ur5_pedestal.urdf.xacro" />

File: robots_ee_pkg/urdf/panda_robot/franka_panda.urdf.xacro (robot description, xacro)
@@ -10,5 +10,5 @@
     <xacro:include filename="$(find robots_ee_pkg)/urdf/panda_robot/panda.gazebo.xacro" />
     <xacro:include filename="$(find robots_ee_pkg)/urdf/panda_robot/panda_hand.transmission.xacro" />
-    <xacro:arg name="hardware_interface" default="PositionJointInterface"/>
+    <xacro:arg name="hardware_interface" default="EffortJointInterface"/>
     <xacro:arg name="gripperHwInterface" default="EffortJointInterface"/>
     <xacro:arg name="arm_name" default="panda"/>

File: robots_ee_pkg/urdf/panda_robot/panda.gazebo.xacro (robot description, xacro)
@@ -12,11 +12,10 @@
       <turnGravityOff>false</turnGravityOff>
       <selfCollide>true</selfCollide>
-      <mu1>0.2</mu1>
-      <mu2>0.2</mu2>
+      <mu1>0.61</mu1>
+      <mu2>0.61</mu2>
     </gazebo>
     <!-- Link1 -->
     <gazebo reference="${arm_name}_link1">
-      <turnGravityOff>false</turnGravityOff>
-      <selfCollide>true</selfCollide>
+      <material>Gazebo/White</material>
       <mu1>0.2</mu1>
       <mu2>0.2</mu2>
@@ -24,6 +23,5 @@
     <!-- Link2 -->
     <gazebo reference="${arm_name}_link2">
-      <turnGravityOff>false</turnGravityOff>
-      <selfCollide>true</selfCollide>
+      <material>Gazebo/White</material>
       <mu1>0.2</mu1>
       <mu2>0.2</mu2>
@@ -31,6 +29,5 @@
     <!-- Link3 -->
     <gazebo reference="${arm_name}_link3">
-      <turnGravityOff>false</turnGravityOff>
-      <selfCollide>true</selfCollide>
+      <material>Gazebo/White</material>
       <mu1>0.2</mu1>
       <mu2>0.2</mu2>
@@ -38,6 +35,5 @@
     <!-- Link4 -->
     <gazebo reference="${arm_name}_link4">
-      <turnGravityOff>false</turnGravityOff>
-      <selfCollide>true</selfCollide>
+      <material>Gazebo/White</material>
       <mu1>0.2</mu1>
       <mu2>0.2</mu2>
@@ -45,6 +41,5 @@
     <!-- Link5 -->
     <gazebo reference="${arm_name}_link5">
-      <turnGravityOff>false</turnGravityOff>
-      <selfCollide>true</selfCollide>
+      <material>Gazebo/White</material>
       <mu1>0.2</mu1>
       <mu2>0.2</mu2>
@@ -52,6 +47,5 @@
     <!-- Link6 -->
     <gazebo reference="${arm_name}_link6">
-      <turnGravityOff>false</turnGravityOff>
-      <selfCollide>true</selfCollide>
+      <material>Gazebo/White</material>>
       <mu1>0.2</mu1>
       <mu2>0.2</mu2>
@@ -59,6 +53,5 @@
     <!-- Link7 -->
     <gazebo reference="${arm_name}_link7">
-      <turnGravityOff>false</turnGravityOff>
-      <selfCollide>true</selfCollide>
+      <material>Gazebo/White</material>
       <mu1>0.2</mu1>
       <mu2>0.2</mu2>

File: robots_ee_pkg/urdf/panda_robot/panda_hand.gazebo.xacro (robot description, xacro)
@@ -4,5 +4,5 @@
     <!-- Link0 -->
     <gazebo reference="${arm_name}_hand">
-      <turnGravityOff>false</turnGravityOff>
+      <material>Gazebo/White</material>
       <mu1>0.2</mu1>
       <mu2>0.2</mu2>
@@ -10,5 +10,5 @@
     <!-- Link1 -->
     <gazebo reference="${arm_name}_leftfinger">
-      <turnGravityOff>false</turnGravityOff>
+      <material>Gazebo/White</material>
       <mu1>0.2</mu1>
       <mu2>0.2</mu2>
@@ -16,5 +16,5 @@
     <!-- Link2 -->
     <gazebo reference="${arm_name}_rightfinger">
-      <turnGravityOff>false</turnGravityOff>
+      <material>Gazebo/White</material>
       <mu1>0.2</mu1>
       <mu2>0.2</mu2>

File: robots_ee_pkg/urdf/panda_robot/panda_system.urdf.xacro (robot description, xacro)
@@ -12,5 +12,18 @@
   <xacro:include filename="$(find robots_ee_pkg)/urdf/panda_robot/franka_panda.urdf.xacro" />
   <xacro:franka_panda_table_urdf table_prefix="$(arg arm_name)" table_parent="$(arg workcell_parent)">
-    <origin xyz="0.5 0 1.0" rpy="0 0 ${pi/2}" />
+    <origin xyz="0 0 1.0" rpy="0 0 0" />
   </xacro:franka_panda_table_urdf>
+  <gazebo reference="world_interface">
+      <gravity>true</gravity>
+  </gazebo>
+  <gazebo>
+      <plugin name="ROSTableControlPlugin" filename="libROSTableControlPlugin.so">
+        <table_cmd_vel>/pand/tbl_cmd_vel</table_cmd_vel>
+        <offset_x>0</offset_x>
+        <offset_y>0</offset_y>
+        <offset_z>1.0</offset_z>
+        <offset_yaw>${pi}</offset_yaw>
+        <table_base_link>iiwa_table_base</table_base_link>
+      </plugin>
+  </gazebo>
 </robot>

Commit message: add panda

File: franka_ros-kinetic-devel/franka_description/robots/hand.xacro (robot description, xacro)
@@ -22,5 +22,5 @@
       <inertial>
         <origin xyz="0 0 0" rpy="0 0 0" />
-        <mass value="0.67893">
+        <mass value="0.67893"/>
         <inertia ixx="0.3" ixy="0.0" ixz="0.0" iyy="0.3" iyz="0.0" izz="0.3" />
       </inertial>
@@ -39,5 +39,5 @@
       <inertial>
         <origin xyz="0 0 0" rpy="0 0 0" />
-        <mass value="0.01053">
+        <mass value="0.01053"/>
         <inertia ixx="0.3" ixy="0.0" ixz="0.0" iyy="0.3" iyz="0.0" izz="0.3" />
       </inertial>
@@ -58,5 +58,5 @@
       <inertial>
         <origin xyz="0 0 0" rpy="0 0 0" />
-        <mass value="0.01053">
+        <mass value="0.01053"/>
         <inertia ixx="0.3" ixy="0.0" ixz="0.0" iyy="0.3" iyz="0.0" izz="0.3" />
       </inertial>

File: franka_ros-kinetic-devel/franka_description/robots/panda_arm.xacro (robot description, xacro)
@@ -8,5 +8,5 @@
         <child link="${arm_id}_link0"/>
         <origin rpy="${rpy}" xyz="${xyz}"/>
-        <dynamic damping="${joint_damping}">
+        <dynamic damping="${joint_damping}"/>
       </joint>
     </xacro:unless>
@@ -24,5 +24,5 @@
       <inertial>
         <origin xyz="0 0 0" rpy="0 0 0" />
-        <mass value="3.06357">
+        <mass value="3.06357"/>
         <inertia ixx="0.3" ixy="0.0" ixz="0.0" iyy="0.3" iyz="0.0" izz="0.3" />
       </inertial>
@@ -41,5 +41,5 @@
       <inertial>
         <origin xyz="0 0 0" rpy="0 0 0" />
-        <mass value="2.34471">
+        <mass value="2.34471"/>
         <inertia ixx="0.3" ixy="0.0" ixz="0.0" iyy="0.3" iyz="0.0" izz="0.3" />
       </inertial>
@@ -66,5 +66,5 @@
       <inertial>
         <origin xyz="0 0 0" rpy="0 0 0" />
-        <mass value="2.36414">
+        <mass value="2.36414"/>
         <inertia ixx="0.3" ixy="0.0" ixz="0.0" iyy="0.3" iyz="0.0" izz="0.3" />
       </inertial>
@@ -91,5 +91,5 @@
       <inertial>
         <origin xyz="0 0 0" rpy="0 0 0" />
-        <mass value="2.38050">
+        <mass value="2.38050"/>
         <inertia ixx="0.3" ixy="0.0" ixz="0.0" iyy="0.3" iyz="0.0" izz="0.3" />
       </inertial>
@@ -116,5 +116,5 @@
       <inertial>
         <origin xyz="0 0 0" rpy="0 0 0" />
-        <mass value="2.42754">
+        <mass value="2.42754"/>
         <inertia ixx="0.3" ixy="0.0" ixz="0.0" iyy="0.3" iyz="0.0" izz="0.3" />
       </inertial>
@@ -141,5 +141,5 @@
       <inertial>
         <origin xyz="0 0 0" rpy="0 0 0" />
-        <mass value="3.49611">
+        <mass value="3.49611"/>
         <inertia ixx="0.3" ixy="0.0" ixz="0.0" iyy="0.3" iyz="0.0" izz="0.3" />
       </inertial>
@@ -166,5 +166,5 @@
       <inertial>
         <origin xyz="0 0 0" rpy="0 0 0" />
-        <mass value="1.46736">
+        <mass value="1.46736"/>
         <inertia ixx="0.3" ixy="0.0" ixz="0.0" iyy="0.3" iyz="0.0" izz="0.3" />
       </inertial>
@@ -191,5 +191,5 @@
       <inertial>
         <origin xyz="0 0 0" rpy="0 0 0" />
-        <mass value="0.45606">
+        <mass value="0.45606"/>
         <inertia ixx="0.3" ixy="0.0" ixz="0.0" iyy="0.3" iyz="0.0" izz="0.3" />
       </inertial>

File: robots_ee_pkg/urdf/iwt_environment.urdf (robot description, URDF)
Before this commit: robot iwt, 33 links, 32 joints
Links:
- removed link iiwa_table_fixed_link
- removed link iiwa_table_x_link
- removed link iiwa_table_yaw_link
- removed link ur5_table_fixed_link
- removed link ur5_table_x_link
- removed link ur5_table_yaw_link
- added link iiwa_table_base, mass 80; collision mesh filename=package://robots_ee_pkg/meshes/lf064_base.stl scale=0.001 0.001 0.001; visual mesh filename=package://robots_ee_pkg/meshes/lf064_base.stl scale=0.001 0.001 0.001
- added link panda_hand, mass 0.67893; collision mesh filename=package://franka_description/meshes/collision/hand.stl; visual mesh filename=package://franka_description/meshes/visual/hand.dae
- added link panda_leftfinger, mass 0.01053; collision mesh filename=package://franka_description/meshes/collision/finger.stl; visual mesh filename=package://franka_description/meshes/visual/finger.dae
- added link panda_link0, mass 3.06357; collision mesh filename=package://franka_description/meshes/collision/link0.stl; visual mesh filename=package://franka_description/meshes/visual/link0.dae
- added link panda_link1, mass 2.34471; collision mesh filename=package://franka_description/meshes/collision/link1.stl; visual mesh filename=package://franka_description/meshes/visual/link1.dae
- added link panda_link2, mass 2.36414; collision mesh filename=package://franka_description/meshes/collision/link2.stl; visual mesh filename=package://franka_description/meshes/visual/link2.dae
- added link panda_link3, mass 2.38050; collision mesh filename=package://franka_description/meshes/collision/link3.stl; visual mesh filename=package://franka_description/meshes/visual/link3.dae
- added link panda_link4, mass 2.42754; collision mesh filename=package://franka_description/meshes/collision/link4.stl; visual mesh filename=package://franka_description/meshes/visual/link4.dae
- added link panda_link5, mass 3.49611; collision mesh filename=package://franka_description/meshes/collision/link5.stl; visual mesh filename=package://franka_description/meshes/visual/link5.dae
- added link panda_link6, mass 1.46736; collision mesh filename=package://franka_description/meshes/collision/link6.stl; visual mesh filename=package://franka_description/meshes/visual/link6.dae
- added link panda_link7, mass 0.45606; collision mesh filename=package://franka_description/meshes/collision/link7.stl; visual mesh filename=package://franka_description/meshes/visual/link7.dae
- added link panda_link8
- added link panda_rightfinger, mass 0.01053; collision mesh filename=package://franka_description/meshes/collision/finger.stl; visual mesh filename=package://franka_description/meshes/visual/finger.dae
- added link panda_table_base, mass 80; collision mesh filename=package://robots_ee_pkg/meshes/lf064_base.stl scale=0.001 0.001 0.001; visual mesh filename=package://robots_ee_pkg/meshes/lf064_base.stl scale=0.001 0.001 0.001
- added link panda_table_ee, mass 20; collision mesh filename=package://robots_ee_pkg/meshes/lf064_table.stl scale=0.001 0.001 0.001; visual mesh filename=package://robots_ee_pkg/meshes/lf064_table.stl scale=0.001 0.001 0.001
- added link ur5_table_base, mass 80; collision mesh filename=package://robots_ee_pkg/meshes/lf064_base.stl scale=0.001 0.001 0.001; visual mesh filename=package://robots_ee_pkg/meshes/lf064_base.stl scale=0.001 0.001 0.001
Joints:
- removed joint iiwa_table_x_joint
- removed joint iiwa_table_yaw_joint
- removed joint ur5_table_x_joint
- removed joint ur5_table_yaw_joint
- added joint panda_finger_joint1: type prismatic, parent panda_hand, child panda_leftfinger, origin xyz=0 0 0.0584 rpy=0 0 0, axis 0 1 0, limit lower=0.0 upper=0.04 effort=20 velocity=0.2
- added joint panda_finger_joint2: type prismatic, parent panda_hand, child panda_rightfinger, origin xyz=0 0 0.0584 rpy=0 0 0, axis 0 -1 0, limit lower=0.0 upper=0.04 effort=20 velocity=0.2, mimic joint=panda_finger_joint1
- added joint panda_hand_joint: type fixed, parent panda_link8, child panda_hand, origin xyz=0 0 0 rpy=0 0 -0.785398163397
- added joint panda_joint1: type revolute, parent panda_link0, child panda_link1, origin xyz=0 0 0.333 rpy=0 0 0, axis 0 0 1, limit lower=-2.8973 upper=2.8973 effort=87 velocity=2.1750
- added joint panda_joint2: type revolute, parent panda_link1, child panda_link2, origin xyz=0 0 0 rpy=-1.57079632679 0 0, axis 0 0 1, limit lower=-1.7628 upper=1.7628 effort=87 velocity=2.1750
- added joint panda_joint3: type revolute, parent panda_link2, child panda_link3, origin xyz=0 -0.316 0 rpy=1.57079632679 0 0, axis 0 0 1, limit lower=-2.8973 upper=2.8973 effort=87 velocity=2.1750
- added joint panda_joint4: type revolute, parent panda_link3, child panda_link4, origin xyz=0.0825 0 0 rpy=1.57079632679 0 0, axis 0 0 1, limit lower=-3.0718 upper=-0.0698 effort=87 velocity=2.1750
- added joint panda_joint5: type revolute, parent panda_link4, child panda_link5, origin xyz=-0.0825 0.384 0 rpy=-1.57079632679 0 0, axis 0 0 1, limit lower=-2.8973 upper=2.8973 effort=12 velocity=2.6100
- added joint panda_joint6: type revolute, parent panda_link5, child panda_link6, origin xyz=0 0 0 rpy=1.57079632679 0 0, axis 0 0 1, limit lower=-0.0175 upper=3.7525 effort=12 velocity=2.6100
- added joint panda_joint7: type revolute, parent panda_link6, child panda_link7, origin xyz=0.088 0 0 rpy=1.57079632679 0 0, axis 0 0 1, limit lower=-2.8973 upper=2.8973 effort=12 velocity=2.6100
- added joint panda_joint8: type fixed, parent panda_link7, child panda_link8, origin xyz=0 0 0.107 rpy=0 0 0, axis 0 0 0
- added joint panda_joint_panda_table_ee: type fixed, parent panda_table_ee, child panda_link0, origin xyz=0 0 0 rpy=0 0 1.57079632679
- added joint panda_table_base_top_joint: type fixed, parent panda_table_base, child panda_table_ee, origin xyz=0.0 0 0.015 rpy=0 0 0
- added joint world_panda_table_joint: type fixed, parent world_interface, child panda_table_base, origin xyz=3.7 -0.5 1.0 rpy=0 0 3.14159265359
- joint iiwa_table_base_top_joint: parent iiwa_table_yaw_link -> iiwa_table_base
- joint ur5_table_base_top_joint: parent ur5_table_yaw_link -> ur5_table_base
- joint world_iiwa_table_joint: child iiwa_table_fixed_link -> iiwa_table_base
- joint world_ur5_table_joint: child ur5_table_fixed_link -> ur5_table_base

File: robots_ee_pkg/urdf/iwt_environment.xacro (robot description, xacro)
@@ -27,5 +27,5 @@
   <xacro:include filename="$(find robots_ee_pkg)/urdf/panda_robot/franka_panda.urdf.xacro" />
   <xacro:franka_panda_table_urdf table_prefix="panda" table_parent="world_interface">
-    <origin xyz="3.7 -0.5 1.0" rpy="0 0 ${pi/2}" />
+    <origin xyz="3.7 -0.5 1.0" rpy="0 0 ${pi}" />
   </xacro:franka_panda_table_urdf>
   <!-- ur5-->

File: robots_ee_pkg/urdf/panda_robot/franka_panda.urdf.xacro (robot description, xacro)
@@ -15,5 +15,5 @@
     <xacro:arg name="robot_param" default="/panda/panda_description"/>
     <xacro:arg name="origin_xyz" default="0 0 0" />
-    <xacro:arg name="origin_rpy" default="0 0 0" />
+    <xacro:arg name="origin_rpy" default="0 0 ${pi/2}" />
     <xacro:arg name="modelDir" default="/home/vishnu/catkin_ws/src/robots_ee_pkg"/>
     <xacro:add_table robot_arm_name="${table_prefix}" table_ee="${table_prefix}_table_ee" modelDir="$(arg modelDir)"  parent="${table_parent}">
@@ -21,7 +21,7 @@
     </xacro:add_table>
     <!-- Panda robot interface -->
-    <xacro:panda_arm  connected_to="${table_prefix}_table_ee" xyz="$(arg origin_xyz)" rpy="$(arg origin_rpy)" />
+    <xacro:panda_arm connected_to="${table_prefix}_table_ee" xyz="$(arg origin_xyz)" rpy="0 0 ${pi/2}" />
     <xacro:panda_gazebo arm_name="$(arg arm_name)" robot_param_name="$(arg robot_param)"/>
-    <xacro:panda_arm_transmission arm_name="$(arg arm_name)" hardware_interface="$(arg hardware_interface)" />
+    <xacro:panda_arm_transmission arm_name="$(arg arm_name)" hardware_interface="EffortJointInterface" />
     <!-- Panda hand interface -->
     <xacro:hand ns="$(arg arm_name)" rpy="0 0 ${-pi/4}" connected_to="$(arg arm_name)_link8" />

File: robots_ee_pkg/urdf/panda_robot/panda.gazebo.xacro (robot description, xacro)
@@ -5,4 +5,5 @@
     <gazebo>
       <plugin name="gazebo_ros_control" filename="libgazebo_ros_control.so">
+      <legacyModeNS>false</legacyModeNS>
         <robotParam>${robot_param_name}</robotParam>
       </plugin>
@@ -10,6 +11,5 @@
     <!-- Link0 -->
     <gazebo reference="${arm_name}_link0">
-      <turnGravityOff>false</turnGravityOff>
-      <selfCollide>true</selfCollide>
+      <material>Gazebo/Grey</material>
       <mu1>0.61</mu1>
       <mu2>0.61</mu2>
@@ -17,5 +17,5 @@
     <!-- Link1 -->
     <gazebo reference="${arm_name}_link1">
-      <material>Gazebo/White</material>
+      <material>Gazebo/Grey</material>
       <mu1>0.2</mu1>
       <mu2>0.2</mu2>
@@ -23,5 +23,5 @@
     <!-- Link2 -->
     <gazebo reference="${arm_name}_link2">
-      <material>Gazebo/White</material>
+      <material>Gazebo/Grey</material>
       <mu1>0.2</mu1>
       <mu2>0.2</mu2>
@@ -29,5 +29,5 @@
     <!-- Link3 -->
     <gazebo reference="${arm_name}_link3">
-      <material>Gazebo/White</material>
+      <material>Gazebo/Grey</material>
       <mu1>0.2</mu1>
       <mu2>0.2</mu2>
@@ -35,5 +35,5 @@
     <!-- Link4 -->
     <gazebo reference="${arm_name}_link4">
-      <material>Gazebo/White</material>
+      <material>Gazebo/Grey</material>
       <mu1>0.2</mu1>
       <mu2>0.2</mu2>
@@ -41,5 +41,5 @@
     <!-- Link5 -->
     <gazebo reference="${arm_name}_link5">
-      <material>Gazebo/White</material>
+      <material>Gazebo/Grey</material>
       <mu1>0.2</mu1>
       <mu2>0.2</mu2>
@@ -47,5 +47,5 @@
     <!-- Link6 -->
     <gazebo reference="${arm_name}_link6">
-      <material>Gazebo/White</material>>
+      <material>Gazebo/Grey</material>>
       <mu1>0.2</mu1>
       <mu2>0.2</mu2>
@@ -53,5 +53,5 @@
     <!-- Link7 -->
     <gazebo reference="${arm_name}_link7">
-      <material>Gazebo/White</material>
+      <material>Gazebo/Grey</material>
       <mu1>0.2</mu1>
       <mu2>0.2</mu2>
