Commit message: table joints

File: robots_ee_pkg/urdf/iwt_environment.urdf (robot description, URDF)
Before this commit: robot iwt, 31 links, 30 joints
Joints:
- removed joint world_iiwa_table_joint
- removed joint world_ur5_table_joint
- added joint iiwa_table_joint: type continuous, parent iiwa_table_base_primary, child iiwa_table_base, origin xyz=0 0 0 rpy=0 0 0, axis 0 0 1
- added joint ur5_table_joint: type continuous, parent ur5_table_base_primary, child ur5_table_base, origin xyz=0 0 0 rpy=0 0 0, axis 0 0 1
- joint world_iiwa_table_primary_x_joint: limit (none) -> lower=-5.0 upper=5.0 effort=10000 velocity=1; type planar -> prismatic
- joint world_ur5_table_primary_x_joint: limit (none) -> lower=-5.0 upper=5.0 effort=10000 velocity=1; type planar -> prismatic

File: robots_ee_pkg/urdf/kuka_robot/kuka_iiwa7.gazebo.xacro (robot description, xacro)
@@ -60,4 +60,11 @@
       <mu2>0.2</mu2>
     </gazebo>
+    <gazebo reference="${robot_name}_table_base_primary">
+      <material>Gazebo/Black</material>
+      <turnGravityOff>true</turnGravityOff>
+      <legacyModeNS>true</legacyModeNS>
+      <mu1>0.1</mu1>
+      <mu2>0.1</mu2>
+    </gazebo>
     <gazebo>
       <plugin name="gazebo_ros_control" filename="libgazebo_ros_control.so">

File: robots_ee_pkg/urdf/table/add_table.urdf.xacro (robot description, xacro)
@@ -6,9 +6,45 @@
         name="add_table">
   <xacro:macro name="add_table" params="robot_arm_name table_ee modelDir parent *origin">
-    <joint name="world_${robot_arm_name}_table_joint" type="fixed">
+    <joint name="world_${robot_arm_name}_table_primary_x_joint" type="prismatic">
       <xacro:insert_block name="origin"/>
       <parent link="${parent}"/>
+      <child link="${robot_arm_name}_table_base_primary"/>
+      <axis xyz="1 0 0" />
+      <limit effort="10000" lower="-5.0" upper="5.0" velocity="1" />
+    </joint>
+    <transmission name="tran1">
+        <type>transmission_interface/SimpleTransmission</type>
+        <joint name="world_${robot_arm_name}_table_primary_x_joint">
+            <hardwareInterface>hardware_interface/EffortJointInterface</hardwareInterface>
+        </joint>
+        <actuator name="motor1">
+            <hardwareInterface>hardware_interface/EffortJointInterface</hardwareInterface>
+            <mechanicalReduction>1</mechanicalReduction>
+        </actuator>
+    </transmission>
+     <joint name="${robot_arm_name}_table_joint" type="continuous">
+      <origin xyz="0 0 0" rpy="0 0 0"/>
+      <parent link="${robot_arm_name}_table_base_primary"/>
       <child link="${robot_arm_name}_table_base"/>
+      <axis xyz="0 0 1" />
     </joint>
+    <transmission name="tran2">
+        <type>transmission_interface/SimpleTransmission</type>
+        <joint name="${robot_arm_name}_table_joint">
+            <hardwareInterface>hardware_interface/EffortJointInterface</hardwareInterface>
+        </joint>
+        <actuator name="motor2">
+            <hardwareInterface>hardware_interface/EffortJointInterface</hardwareInterface>
+            <mechanicalReduction>1</mechanicalReduction>
+        </actuator>
+    </transmission>
+    <link name="${robot_arm_name}_table_base_primary" />
+    <gazebo reference="${robot_arm_name}_table_base_primary">
+      <material>Gazebo/Black</material>
+      <turnGravityOff>true</turnGravityOff>
+      <legacyModeNS>true</legacyModeNS>
+      <mu1>0.5</mu1>
+      <mu2>0.4</mu2>
+    </gazebo>
      <!-- BASE LINK -->
     <link name="${robot_arm_name}_table_base">

Commit message: table link changes- do not pull from PC until every...

File: robots_ee_pkg/urdf/iwt_environment.urdf (robot description, URDF)
Before this commit: robot iwt, 31 links, 30 joints
Links:
- removed link iiwa_table_base
- removed link iiwa_table_base_primary
- removed link ur5_table_base
- removed link ur5_table_base_primary
- added link iiwa_table_fixed_link, mass 1; visual box size=0.001 0.001 0.001
- added link iiwa_table_x_link, mass 1; visual box size=0.001 0.001 0.001
- added link iiwa_table_yaw_link, mass 80; collision mesh filename=package://robots_ee_pkg/meshes/lf064_base.stl scale=0.001 0.001 0.001; visual mesh filename=package://robots_ee_pkg/meshes/lf064_base.stl scale=0.001 0.001 0.001
- added link ur5_table_fixed_link, mass 1; visual box size=0.001 0.001 0.001
- added link ur5_table_x_link, mass 1; visual box size=0.001 0.001 0.001
- added link ur5_table_yaw_link, mass 80; collision mesh filename=package://robots_ee_pkg/meshes/lf064_base.stl scale=0.001 0.001 0.001; visual mesh filename=package://robots_ee_pkg/meshes/lf064_base.stl scale=0.001 0.001 0.001
Joints:
- removed joint iiwa_table_joint
- removed joint ur5_table_joint
- removed joint world_iiwa_table_primary_x_joint
- removed joint world_ur5_table_primary_x_joint
- added joint iiwa_table_x_joint: type prismatic, parent iiwa_table_fixed_link, child iiwa_table_x_link, origin xyz=0 0 0 rpy=0 0 0, axis 1 0 0, limit lower=-5.0 upper=5.0 effort=10000 velocity=1
- added joint iiwa_table_yaw_joint: type continuous, parent iiwa_table_x_link, child iiwa_table_yaw_link, origin xyz=0 0 0 rpy=0 0 0, axis 0 0 1
- added joint ur5_table_x_joint: type prismatic, parent ur5_table_fixed_link, child ur5_table_x_link, origin xyz=0 0 0 rpy=0 0 0, axis 1 0 0, limit lower=-5.0 upper=5.0 effort=10000 velocity=1
- added joint ur5_table_yaw_joint: type continuous, parent ur5_table_x_link, child ur5_table_yaw_link, origin xyz=0 0 0 rpy=0 0 0, axis 0 0 1
- added joint world_iiwa_table_joint: type fixed, parent world_interface, child iiwa_table_fixed_link, origin xyz=2.25 -0.5 1.0 rpy=0 0 3.14159265359
- added joint world_ur5_table_joint: type fixed, parent world_interface, child ur5_table_fixed_link, origin xyz=0.8 -0.5 1.0 rpy=0 0 3.14159265359
- joint iiwa_table_base_top_joint: parent iiwa_table_base -> iiwa_table_yaw_link
- joint ur5_table_base_top_joint: parent ur5_table_base -> ur5_table_yaw_link

File: robots_ee_pkg/urdf/table/add_table.urdf.xacro (robot description, xacro)
@@ -9,8 +9,54 @@
       <xacro:insert_block name="origin"/>
       <parent link="${parent}"/>
-      <child link="${robot_arm_name}_table_base"/>
+      <child link="${robot_arm_name}_table_fixed_link"/>
     </joint>
+    <joint name="${robot_arm_name}_table_x_joint" type="prismatic">
+      <origin xyz="0 0 0" rpy="0 0 0"/>
+      <parent link="${robot_arm_name}_table_fixed_link"/>
+      <child link="${robot_arm_name}_table_x_link"/>
+      <axis xyz="1 0 0" />
+      <limit effort="10000" lower="-5.0" upper="5.0" velocity="1" />
+    </joint>
+    <joint name="${robot_arm_name}_table_yaw_joint" type="continuous">
+      <origin xyz="0 0 0" rpy="0 0 0"/>
+      <parent link="${robot_arm_name}_table_x_link"/>
+      <child link="${robot_arm_name}_table_yaw_link"/>
+      <axis xyz="0 0 1" />
+    </joint>
+    <!-- Extra links-->
+    <link name="${robot_arm_name}_table_fixed_link">
+      <inertial>
+        <mass value="1"/>
+          <origin xyz="0 0 0" />
+            <inertia  ixx="1" ixy="0.0"  ixz="0.0"  iyy="1"  iyz="0.0"  izz="1" />
+      </inertial>
+     <visual>
+        <origin rpy="0 0 0" xyz="0.0 0 0"/>
+        <geometry>
+          <box size="0.001 0.001 0.001" />
+        </geometry>
+        <material name="grey">
+          <color rgba="0.5 0.5 0.5 1"/>
+        </material>
+      </visual>
+    </link>
+    <link name="${robot_arm_name}_table_x_link" >
+      <inertial>
+        <mass value="1"/>
+          <origin xyz="0 0 0" />
+            <inertia  ixx="1" ixy="0.0"  ixz="0.0"  iyy="1"  iyz="0.0"  izz="1" />
+      </inertial>
+     <visual>
+        <origin rpy="0 0 0" xyz="0.0 0 0"/>
+        <geometry>
+          <box size="0.001 0.001 0.001" />
+        </geometry>
+        <material name="grey">
+          <color rgba="0.5 0.5 0.5 1"/>
+        </material>
+      </visual>
+    </link>
      <!-- BASE LINK -->
-    <link name="${robot_arm_name}_table_base">
+    <link name="${robot_arm_name}_table_yaw_link">
       <inertial>
         <mass value="80"/>
@@ -35,5 +81,5 @@
       </collision>
     </link>
-    <gazebo reference="${robot_arm_name}_table_base">
+    <gazebo reference="${robot_arm_name}_table_yaw_link">
       <material>Gazebo/Grey</material>
       <turnGravityOff>true</turnGravityOff>
@@ -43,5 +89,5 @@
     <joint name="${robot_arm_name}_table_base_top_joint" type="fixed">
       <origin rpy="0 0 0" xyz="0.0 0 0.015"/>
-      <parent link="${robot_arm_name}_table_base"/>
+      <parent link="${robot_arm_name}_table_yaw_link"/>
       <child link="${table_ee}"/>
     </joint>
@@ -76,4 +122,38 @@
       <mu2>0.4</mu2>
     </gazebo>
+    <gazebo reference="${robot_arm_name}_table_fixed_link">
+      <material>Gazebo/Grey</material>
+      <selfCollide>false</selfCollide>
+      <turnGravityOff>true</turnGravityOff>
+      <mu1>0.1</mu1>
+      <mu2>0.1</mu2>
+    </gazebo>
+    <gazebo reference="${robot_arm_name}_table_x_link">
+      <material>Gazebo/Grey</material>
+      <selfCollide>false</selfCollide>
+      <turnGravityOff>true</turnGravityOff>
+      <mu1>0.1</mu1>
+      <mu2>0.1</mu2>
+    </gazebo>
+    <transmission name="tran1">
+        <type>transmission_interface/SimpleTransmission</type>
+        <joint name="${robot_arm_name}_table_x_joint">
+            <hardwareInterface>hardware_interface/EffortJointInterface</hardwareInterface>
+        </joint>
+        <actuator name="motor1">
+            <hardwareInterface>hardware_interface/EffortJointInterface</hardwareInterface>
+            <mechanicalReduction>1</mechanicalReduction>
+        </actuator>
+    </transmission>
+    <transmission name="tran2">
+        <type>transmission_interface/SimpleTransmission</type>
+        <joint name="${robot_arm_name}_table_yaw_joint">
+            <hardwareInterface>hardware_interface/EffortJointInterface</hardwareInterface>
+        </joint>
+        <actuator name="motor2">
+            <hardwareInterface>hardware_interface/EffortJointInterface</hardwareInterface>
+            <mechanicalReduction>1</mechanicalReduction>
+        </actuator>
+    </transmission>
   </xacro:macro>
 </robot>

Commit message: Panda seperate description for Gazebo simulation

File: robots_ee_pkg/urdf/iwt_environment.urdf (robot description, URDF)
Before this commit: robot iwt, 43 links, 42 joints
Links:
- link panda_hand: geometry collision mesh filename=package://robots_ee_pkg/meshes/collision/hand.stl; visual mesh filename=package://robots_ee_pkg/meshes/visual/hand.dae
- link panda_leftfinger: geometry collision mesh filename=package://robots_ee_pkg/meshes/collision/finger.stl; visual mesh filename=package://robots_ee_pkg/meshes/visual/finger.dae
- link panda_link0: geometry collision mesh filename=package://robots_ee_pkg/meshes/collision/link0.stl; visual mesh filename=package://robots_ee_pkg/meshes/visual/link0.dae
- link panda_link1: geometry collision mesh filename=package://robots_ee_pkg/meshes/collision/link1.stl; visual mesh filename=package://robots_ee_pkg/meshes/visual/link1.dae
- link panda_link2: geometry collision mesh filename=package://robots_ee_pkg/meshes/collision/link2.stl; visual mesh filename=package://robots_ee_pkg/meshes/visual/link2.dae
- link panda_link3: geometry collision mesh filename=package://robots_ee_pkg/meshes/collision/link3.stl; visual mesh filename=package://robots_ee_pkg/meshes/visual/link3.dae
- link panda_link4: geometry collision mesh filename=package://robots_ee_pkg/meshes/collision/link4.stl; visual mesh filename=package://robots_ee_pkg/meshes/visual/link4.dae
- link panda_link5: geometry collision mesh filename=package://robots_ee_pkg/meshes/collision/link5.stl; visual mesh filename=package://robots_ee_pkg/meshes/visual/link5.dae
- link panda_link6: geometry collision mesh filename=package://robots_ee_pkg/meshes/collision/link6.stl; visual mesh filename=package://robots_ee_pkg/meshes/visual/link6.dae
- link panda_link7: geometry collision mesh filename=package://robots_ee_pkg/meshes/collision/link7.stl; visual mesh filename=package://robots_ee_pkg/meshes/visual/link7.dae
- link panda_rightfinger: geometry collision mesh filename=package://robots_ee_pkg/meshes/collision/finger.stl; visual mesh filename=package://robots_ee_pkg/meshes/visual/finger.dae

File: robots_ee_pkg/urdf/panda_robot/franka_panda.urdf.xacro (robot description, xacro)
@@ -4,6 +4,6 @@
   <xacro:macro name = "franka_panda_table_urdf" params = "table_prefix table_parent *origin">
     <!--Import the lbr iiwa macro -->
-    <xacro:include filename="$(find franka_description)/robots/panda_arm.xacro"/>
-    <xacro:include filename="$(find franka_description)/robots/hand.xacro"/>
+    <xacro:include filename="$(find robots_ee_pkg)/urdf/panda_robot/robots/panda_arm.xacro"/>
+    <xacro:include filename="$(find robots_ee_pkg)/urdf/panda_robot/robots/hand.xacro"/>
     <xacro:include filename="$(find robots_ee_pkg)/urdf/table/add_table.urdf.xacro" />
     <xacro:include filename="$(find robots_ee_pkg)/urdf/panda_robot/panda.transmission.xacro" />
