Commit message: omron fake laser

File: omronld/omronld_description/urdf/laser/sick_lms1xx.urdf.xacro (robot description, xacro)
@@ -1,6 +1,6 @@
 <?xml version="1.0"?>
 <robot xmlns:xacro="http://ros.org/wiki/xacro">
-  <xacro:macro name="sick_lms1xx" params="frame:=laser topic:=scan sample_size:=720 update_rate:=50
-               min_angle:=-2.0944 max_angle:=2.0944 min_range:=0.1 max_range:=15 robot_description:=/" >
+  <xacro:macro name="sick_lms1xx" params="frame:=laser parent:=base_link topic:=scan sample_size:=720 update_rate:=50
+               min_angle:=-2.0944 max_angle:=2.0944 min_range:=0.1 max_range:=15 robot_description:=/ *origin" >
     <link name="${frame}">
       <inertial>
@@ -25,8 +25,8 @@
       </collision>
     </link>
-    <joint name="laser_joint" type="fixed">
-      <origin xyz="$(arg laser_xyz)" rpy="$(arg laser_rpy)" />
-      <parent link="base_link" />
-      <child link="base_laser" />
+    <joint name="${frame}_joint" type="fixed">
+      <xacro:insert_block name="origin"/>
+      <parent link="${parent}" />
+      <child link="${frame}" />
     </joint>
     <gazebo reference="${frame}">
@@ -34,5 +34,5 @@
       <sensor type="ray" name="${frame}">
         <pose>0 0 0 0 0 0</pose>
-        <visualize>false</visualize>
+        <visualize>true</visualize>
         <update_rate>${update_rate}</update_rate>
         <ray>

File: omronld/omronld_description/urdf/omronld.urdf (robot description, URDF)
Before this commit: robot omronld, 8 links, 7 joints
Links:
- added link base_laser_fake, mass 1.1; collision box size=0.105 0.1 0.1; visual mesh filename=package://omronld_description/meshes/laser/sick-lms1xx.dae
Joints:
- removed joint laser_joint
- added joint base_laser_fake_joint: type fixed, parent base_link, child base_laser_fake, origin xyz=-0.2652 0.0 0.201 rpy=-3.14159 0.0 0.0
- added joint base_laser_joint: type fixed, parent base_link, child base_laser, origin xyz=0.2652 0.0 0.201 rpy=3.14159 0.0 0.0

File: omronld/omronld_description/urdf/omronld.urdf.xacro (robot description, xacro)
@@ -17,6 +17,4 @@
   <!-- LASER -->
   <xacro:include filename="$(find omronld_description)/urdf/laser/sick_lms1xx.urdf.xacro" />
-  <xacro:arg name="laser_xyz" default="$(optenv omronld_LMS1XX_XYZ 0.2652 0.0 0.201)" />
-  <xacro:arg name="laser_rpy" default="$(optenv omronld_LMS1XX_RPY ${M_PI} 0.0 0.0)" />
   <!-- base_link origin point is center of rotation, on the floor. -->
   <link name="base_link">
@@ -46,5 +44,10 @@
   </xacro:omronld_wheel>
   <!-- LASER -->
-  <xacro:sick_lms1xx frame="base_laser" topic="scan" robot_description="/"/> <!-- <xacro: muesste man hier nicht mit anfuegen funktioniert auch ohne-->
+  <xacro:sick_lms1xx frame="base_laser" parent="base_link" topic="scan">
+    <origin xyz="0.2652 0.0 0.201" rpy="${M_PI} 0.0 0.0"/>
+  </xacro:sick_lms1xx>
+  <xacro:sick_lms1xx frame="base_laser_fake" parent="base_link" topic="scanFake">
+    <origin xyz="-0.2652 0.0 0.201" rpy="${-M_PI} 0.0 0.0"/>
+  </xacro:sick_lms1xx>
   <!-- GAZEBO PLUGINS--> <!-- http://wiki.ros.org/urdf/Tutorials/Using%20a%20URDF%20in%20Gazebo-->
   <gazebo>
