Commit message: gazebo erroe correction

File: omronld/omronld_description/urdf/omronld.urdf.xacro (robot description, xacro)
@@ -50,4 +50,5 @@
   <gazebo>
     <plugin name="gazebo_ros_control" filename="libgazebo_ros_control.so">
+      <legacyModeNS>false</legacyModeNS>
       <robotParam>/$(arg robot_description)</robotParam>
     </plugin>

File: robots_ee_pkg/urdf/kuka_robot/kuka_iiwa7.gazebo.xacro (robot description, xacro)
@@ -63,4 +63,5 @@
       <plugin name="gazebo_ros_control" filename="libgazebo_ros_control.so">
         <robotParam>${robot_parameter_name}</robotParam>
+        <legacyModeNS>false</legacyModeNS>
       </plugin>
     </gazebo>

File: robots_ee_pkg/urdf/table/add_table.urdf.xacro (robot description, xacro)
@@ -6,45 +6,9 @@
         name="add_table">
   <xacro:macro name="add_table" params="robot_arm_name table_ee modelDir parent *origin">
-    <joint name="world_${robot_arm_name}_table_primary_x_joint" type="prismatic">
+    <joint name="world_${robot_arm_name}_table_joint" type="fixed">
       <xacro:insert_block name="origin"/>
       <parent link="${parent}"/>
-      <child link="${robot_arm_name}_table_base_primary"/>
-      <axis xyz="1 0 0" />
-      <limit effort="10000" lower="-5.0" upper="5.0" velocity="1" />
+      <child link="${robot_arm_name}_table_base"/>
     </joint>
-    <transmission name="tran1">
-        <type>transmission_interface/SimpleTransmission</type>
-        <joint name="world_${robot_arm_name}_table_primary_x_joint">
-            <hardwareInterface>hardware_interface/EffortJointInterface</hardwareInterface>
-        </joint>
-        <actuator name="motor1">
-            <hardwareInterface>hardware_interface/EffortJointInterface</hardwareInterface>
-            <mechanicalReduction>1</mechanicalReduction>
-        </actuator>
-    </transmission>
-     <joint name="${robot_arm_name}_table_joint" type="continuous">
-      <origin xyz="0 0 0" rpy="0 0 0"/>
-      <parent link="${robot_arm_name}_table_base_primary"/>
-      <child link="${robot_arm_name}_table_base"/>
-      <axis xyz="0 0 1" />
-    </joint>
-    <transmission name="tran2">
-        <type>transmission_interface/SimpleTransmission</type>
-        <joint name="${robot_arm_name}_table_joint">
-            <hardwareInterface>hardware_interface/EffortJointInterface</hardwareInterface>
-        </joint>
-        <actuator name="motor2">
-            <hardwareInterface>hardware_interface/EffortJointInterface</hardwareInterface>
-            <mechanicalReduction>1</mechanicalReduction>
-        </actuator>
-    </transmission>
-    <link name="${robot_arm_name}_table_base_primary" />
-    <gazebo reference="${robot_arm_name}_table_base_primary">
-      <material>Gazebo/Black</material>
-      <turnGravityOff>true</turnGravityOff>
-      <legacyModeNS>true</legacyModeNS>
-      <mu1>0.5</mu1>
-      <mu2>0.4</mu2>
-    </gazebo>
      <!-- BASE LINK -->
     <link name="${robot_arm_name}_table_base">

File: robots_ee_pkg/urdf/ur5_robot/ur5.gazebo.xacro (robot description, xacro)
@@ -34,4 +34,5 @@
       <plugin name="gazebo_ros_control" filename="libgazebo_ros_control.so">
         <robotParam>${robot_parameter_name}</robotParam>
+        <legacyModeNS>false</legacyModeNS>
       </plugin>
     </gazebo>

Commit message: omron update after test

File: omronld/omronld_description/urdf/omronld.urdf.xacro (robot description, xacro)
@@ -31,5 +31,5 @@
     <collision name="base_link_collision">
       <geometry name="base_link_collision_geom">
-        <box size="0.7 0.5 0.05" />
+        <box size="0.7 0.5 0.001" />
       </geometry>
       <origin xyz="0 0 0.1" rpy="0 0 0" />
@@ -48,5 +48,5 @@
   </xacro:sick_lms1xx>
   <xacro:sick_lms1xx frame="base_laser_fake" parent="base_link" topic="scanFake">
-    <origin xyz="-0.2652 0.0 0.201" rpy="${-M_PI} 0.0 0.0"/>
+    <origin xyz="-0.2652 0.0 0.105" rpy="${M_PI} 0.0 ${M_PI}"/>
   </xacro:sick_lms1xx>
   <!-- GAZEBO PLUGINS--> <!-- http://wiki.ros.org/urdf/Tutorials/Using%20a%20URDF%20in%20Gazebo-->
