Commit message: new spawn stactic tf2 update

File: iwtros_descriptions/robots_ee_pkg/urdf/kuka_robot/kuka_iiwa7_system.urdf.xacro (robot description, xacro)
@@ -7,5 +7,5 @@
   <xacro:arg name="robot_param" default="/iiwa/iiwa_description"/>
   <xacro:arg name="workcell_parent" default="world_interface"/>
-  <link name="world_interface"/>
+  <link name="$(arg workcell_parent)"/>
   <!-- origin is given as in the iwt_envirnment.xacro for urdf
         If any changes requred int the position of the the system change it according to the iwt_envirnment.xacro -->
@@ -14,5 +14,5 @@
     <origin xyz="0 0 1.0" rpy="0 0 0" />
   </xacro:kuka_iiwa7_table_urdf>
-  <gazebo reference="world_interface">
+  <gazebo reference="$(arg workcell_parent)">
       <gravity>true</gravity>
   </gazebo>

File: iwtros_descriptions/robots_ee_pkg/urdf/panda_robot/panda_system.urdf.xacro (robot description, xacro)
@@ -7,5 +7,5 @@
   <xacro:arg name="robot_param" default="/panda/panda_description"/>
   <xacro:arg name="workcell_parent" default="world_interface"/>
-  <link name="world_interface"/>
+  <link name="$(arg workcell_parent)"/>
   <!-- origin is given as in the iwt_envirnment.xacro for urdf
         If any changes requred int the position of the the system change it according to the iwt_envirnment.xacro -->
@@ -14,5 +14,5 @@
     <origin xyz="0 0 1.0" rpy="0 0 0" />
   </xacro:franka_panda_table_urdf>
-  <gazebo reference="world_interface">
+  <gazebo reference="$(arg workcell_parent)">
       <gravity>true</gravity>
   </gazebo>

File: iwtros_descriptions/robots_ee_pkg/urdf/ur5_robot/ur5_system.urdf.xacro (robot description, xacro)
@@ -4,5 +4,5 @@
   <xacro:arg name="robot_param" default="/ur5/ur5_description"/>
   <xacro:arg name="workcell_parent" default="world_interface"/>
-  <link name="world_interface"/>
+  <link name="$(arg workcell_parent)"/>
   <!-- origin is given as in the iwt_envirnment.xacro for urdf -->
   <xacro:include filename="$(find robots_ee_pkg)/urdf/ur5_robot/ur5_pedestal.urdf.xacro" />
@@ -10,5 +10,5 @@
     <origin xyz="0 0 1.0" rpy="0 0 0" />
   </xacro:ur5_table_urdf>
-  <gazebo reference="world_interface">
+  <gazebo reference="$(arg workcell_parent)">
     <gravity>true</gravity>
   </gazebo>
