Commit message: Updated wsg50 package
Setting update


KUKA urdf update

File: iwtros_descriptions/robots_ee_pkg/urdf/kuka_robot/kuka_iiwa7.urdf.xacro (robot description, xacro)
@@ -29,5 +29,5 @@
   <xacro:iiwa_system_gazebo robot_name="$(arg robot_name)" robot_parameter_name="$(arg robot_param)"/>
   <!-- schunck greifer -->
-  <xacro:wsg_50_xacro name="wsg50" parent="$(arg robot_name)_link_ee" gripperHwInterface="$(arg gripperHwInterface)">
+  <xacro:wsg_50_xacro name="wsg50" parent="$(arg robot_name)_link_ee" finger_length="0.023" finger_tip="0">
     <origin xyz="0 0 0" rpy="0 0 0" />
   </xacro:wsg_50_xacro>

File: wsg50-ros-pkg/wsg_50_simulation/urdf/wsg_50.urdf.xacro (robot description, xacro)
@@ -3,12 +3,12 @@
 	xmlns:controller="http://playerstage.sourceforge.net/gazebo/xmlschema/#controller"
 	xmlns:interface="http://playerstage.sourceforge.net/gazebo/xmlschema/#interface"
-        xmlns:xacro="http://www.ros.org/wiki/xacro"
+        xmlns:xacro="http://ros.org/wiki/xacro"
 	name="wsg_50">
 <!-- finger_length: Length of finger from gripper base. (was 0.023) -->
 <!-- finger_tip:    Offset of finger tip along fingers' motion direction.
                     Use e.g. for single contact point tip on finger. (default 0) -->
-<xacro:macro name="wsg_50_xacro" params="name parent gripperHwInterface *origin">
+<xacro:macro name="wsg_50_xacro" params="name parent finger_length finger_tip *origin">
  <joint name="${name}_anterior_gripper_joint" type="fixed">
-    <xacro:insert_block name="origin"/>
+    <insert_block name="origin"/>
     <parent link="${parent}"/>
     <child link="${name}_base_link"/>
@@ -17,5 +17,5 @@
  <link name="${name}_base_link">
       <inertial>
-          <mass value="1.15"/>
+          <mass value="0.25" />
           <origin xyz="0 0 0" />
      	  <!--inertia ixx="1.0" ixy="0.0" ixz="0.0"
@@ -46,24 +46,26 @@
     <turnGravityOff>false</turnGravityOff>
   </gazebo>
+  <joint name="${name}_center_joint" type="fixed">
+     <origin xyz="0 0 ${finger_length}" rpy="0 0 0" />      <!--origin xyz="-0.0067 0 0.049" rpy="0 0 0" /-->
+     <parent link="${name}_base_link"/>
+     <child link="${name}_center" />
+  </joint>
+  <link name="${name}_center">
+  </link>
   <!-- GRIPPER LEFT -->
-  <joint name="${name}_gripper_left_joint" type="prismatic">
+  <joint name="${name}_finger_left_joint" type="prismatic">
      <limit lower="-0.055" upper="-0.0027" effort="1.0" velocity="1.0"/>
      <origin xyz="0 0 0" rpy="0 0 0" />      <!--origin xyz="-0.0067 0 0.049" rpy="0 0 0" /-->
      <parent link="${name}_base_link"/>
      <child link="${name}_gripper_left" />
-     <dynamics friction="0.1" damping="0.1" />
+     <dynamics friction="100" damping="100" />
      <axis xyz="1 0 0"/>
      <limit effort="100" velocity="100"/>
   </joint>
-  <transmission name="${name}_base_trans_left">
-     <type>transmission_interface/SimpleTransmission</type>
-     <actuator name="${name}_base_motor_left">
-       <hardwareInterface>hardware_interface/${gripperHwInterface}</hardwareInterface>
-       <mechanicalReduction>1</mechanicalReduction>
-       <!--motorTorqueConstant>1</motorTorqueConstant-->
-     </actuator>
-     <joint name="${name}_gripper_left_joint">
-      <hardwareInterface>hardware_interface/${gripperHwInterface}</hardwareInterface>
-     </joint>
+  <transmission name="${name}_base_trans_left" type="pr2_mechanism_model/SimpleTransmission">
+     <actuator name="${name}_base_motor_left" />
+     <joint name="${name}_base_joint_gripper_left" />
+     <mechanicalReduction>1</mechanicalReduction>
+     <motorTorqueConstant>1</motorTorqueConstant>
   </transmission>
   <link name="${name}_gripper_left">
@@ -78,16 +80,16 @@
           <origin xyz="0.0 0 0" rpy="0 0 0" />
           <geometry>
-             <mesh filename="package://wsg_50_simulation/meshes/GUIDE_WSG50_110.dae" scale="0.001 0.001 0.001"/>
-	     <!--box size="0.0175 0.03 0.024"/-->
-          </geometry>
-          <material name="black">
-		<color rgba="0 0 0 0"/>
-      	  </material>
-      </visual>
-      <collision>
-          <origin xyz="0 0 0" rpy="0 0 0" />
-          <geometry>
-	     <!--box size="0.0175 0.03 0.024"/-->
-             <mesh filename="package://wsg_50_simulation/meshes/GUIDE_WSG50_110.dae" scale="0.001 0.001 0.001"/>
+             <mesh filename="package://wsg_50_simulation/meshes/GUIDE_WSG50_110.stl" scale="0.001 0.001 0.001"/>
+	     <!--box size="0.0175 0.03 0.024"/-->
+          </geometry>
+          <material name="black">
+		<color rgba="0 0 0 0"/>
+      	  </material>
+      </visual>
+      <collision>
+          <origin xyz="0 0 0" rpy="0 0 0" />
+          <geometry>
+	     <!--box size="0.0175 0.03 0.024"/-->
+             <mesh filename="package://wsg_50_simulation/meshes/GUIDE_WSG50_110.stl" scale="0.001 0.001 0.001"/>
          </geometry>
      </collision>
@@ -98,6 +100,44 @@
     <turnGravityOff>false</turnGravityOff>
   </gazebo>
+  <!-- LEFT FINGER -->
+  <joint name="${name}_guide_joint_finger_left" type="fixed">
+     <origin xyz="${finger_tip} 0 ${finger_length}" rpy="0 0 0" />
+     <parent link="${name}_gripper_left"/>
+     <child link="${name}_finger_left" />
+     <dynamics friction="100" damping="100" />
+     <axis xyz="1 0 0"/>
+     <limit effort="100" velocity="100"/>
+  </joint>
+  <link name="${name}_finger_left">
+      <inertial>
+          <mass value="0.1" />
+          <origin xyz="0 0 0" />
+      <inertia ixx="1.0" ixy="0.0" ixz="0.0"
+               iyy="1.0" iyz="0.0"
+               izz="1.0" />
+      </inertial>
+      <visual>
+          <origin xyz="0.0 0 0" rpy="0 0 0" />
+          <geometry>
+             <mesh filename="package://wsg_50_simulation/meshes/WSG-FMF.stl" scale="0.001 0.001 0.001"/>
+          </geometry>
+          <material name="black">
+		<color rgba="0 0 0 0"/>
+      	  </material>
+      </visual>
+      <collision>
+          <origin xyz="0 0 0" rpy="0 0 0" />
+          <geometry>
+             <mesh filename="package://wsg_50_simulation/meshes/WSG-FMF.stl" scale="0.001 0.001 0.001"/>
+         </geometry>
+     </collision>
+     <contact_coefficients kd="1.0" kp="1000.0" mu="0"/>
+  </link>
+  <gazebo reference="${name}_finger_left">
+    <material>Gazebo/Blue</material>
+    <turnGravityOff>false</turnGravityOff>
+  </gazebo>
   <!-- GRIPPER RIGHT -->
-  <joint name="${name}_gripper_right_joint" type="prismatic">
+  <joint name="${name}_finger_right_joint" type="prismatic">
      <limit lower="0.0027" upper="0.055" effort="1.0" velocity="1.0"/>
      <origin xyz="0 0 0" rpy="0 0 3.14159" />
@@ -105,17 +145,12 @@
      <child link="${name}_gripper_right" />
      <axis xyz="-1 0 0"/>
-     <dynamics friction="0.1" damping="0.1" />
-     <limit effort="100" velocity="100"/>
-  </joint>
-  <transmission name="${name}_base_trans_right">
-     <type>transmission_interface/SimpleTransmission</type>
-     <actuator name="${name}_base_motor_right">
-        <hardwareInterface>hardware_interface/${gripperHwInterface}</hardwareInterface>
-        <mechanicalReduction>1</mechanicalReduction>
-       <!--motorTorqueConstant>1</motorTorqueConstant-->
-     </actuator>
-     <joint name="${name}_gripper_right_joint">
-        <hardwareInterface>hardware_interface/${gripperHwInterface}</hardwareInterface>
-     </joint>
+     <dynamics friction="100" damping="100" />
+     <limit effort="100" velocity="100"/>
+  </joint>
+  <transmission name="${name}_base_trans_right" type="pr2_mechanism_model/SimpleTransmission">
+     <actuator name="${name}_base_motor_right" />
+     <joint name="${name}_base_joint_gripper_right" />
+     <mechanicalReduction>1</mechanicalReduction>
+     <motorTorqueConstant>1</motorTorqueConstant>
   </transmission>
     <link name="${name}_gripper_right">
@@ -130,16 +165,16 @@
           <origin xyz="0.0 0 0" rpy="0 0 0" />
           <geometry>
-             <mesh filename="package://wsg_50_simulation/meshes/GUIDE_WSG50_110.dae" scale="0.001 0.001 0.001"/>
-	     <!--box size="0.0175 0.03 0.024"/-->
-          </geometry>
-          <material name="black">
-		<color rgba="0 0 0 0"/>
-      	  </material>
-      </visual>
-      <collision>
-          <origin xyz="0 0 0" rpy="0 0 0" />
-          <geometry>
-	     <!--box size="0.0175 0.03 0.024"/-->
-             <mesh filename="package://wsg_50_simulation/meshes/GUIDE_WSG50_110.dae" scale="0.001 0.001 0.001"/>
+             <mesh filename="package://wsg_50_simulation/meshes/GUIDE_WSG50_110.stl" scale="0.001 0.001 0.001"/>
+	     <!--box size="0.0175 0.03 0.024"/-->
+          </geometry>
+          <material name="black">
+		<color rgba="0 0 0 0"/>
+      	  </material>
+      </visual>
+      <collision>
+          <origin xyz="0 0 0" rpy="0 0 0" />
+          <geometry>
+	     <!--box size="0.0175 0.03 0.024"/-->
+             <mesh filename="package://wsg_50_simulation/meshes/GUIDE_WSG50_110.stl" scale="0.001 0.001 0.001"/>
          </geometry>
      </collision>
@@ -150,16 +185,42 @@
     <turnGravityOff>false</turnGravityOff>
   </gazebo>
-<!-- <gazebo>
-  <plugin name="gazebo_ros_control" filename="libgazebo_ros_control.so">
-    <robotNamespace>/</robotNamespace>
-  </plugin>
-</gazebo>
-  <gazebo>
-    <controller:gazebo_ros_controller_manager name="gazebo_ros_controller_manager" plugin="libgazebo_ros_controller_manager.so">
-      <alwaysOn>true</alwaysOn>
-      <updateRate>1000.0</updateRate>
-      <interface:audio name="gazebo_ros_controller_manager_dummy_iface" />
-    </controller:gazebo_ros_controller_manager>
-  </gazebo> -->
+  <!-- RIGHT FINGER -->
+  <joint name="${name}_guide_joint_finger_right" type="fixed">
+     <origin xyz="${finger_tip} 0 ${finger_length}" rpy="0 0 0" />
+     <parent link="${name}_gripper_right"/>
+     <child link="${name}_finger_right" />
+     <dynamics friction="100" damping="100" />
+     <axis xyz="1 0 0"/>
+     <limit effort="100" velocity="100"/>
+  </joint>
+  <link name="${name}_finger_right">
+      <inertial>
+          <mass value="0.1" />
+          <origin xyz="0 0 0" />
+      <inertia ixx="1.0" ixy="0.0" ixz="0.0"
+               iyy="1.0" iyz="0.0"
+               izz="1.0" />
+      </inertial>
+      <visual>
+          <origin xyz="0.0 0 0" rpy="0 0 0" />
+          <geometry>
+             <mesh filename="package://wsg_50_simulation/meshes/WSG-FMF.stl" scale="0.001 0.001 0.001"/>
+          </geometry>
+          <material name="black">
+		<color rgba="0 0 0 0"/>
+      	  </material>
+      </visual>
+      <collision>
+          <origin xyz="0 0 0" rpy="0 0 0" />
+          <geometry>
+             <mesh filename="package://wsg_50_simulation/meshes/WSG-FMF.stl" scale="0.001 0.001 0.001"/>
+         </geometry>
+     </collision>
+     <contact_coefficients kd="1.0" kp="1000.0" mu="0"/>
+  </link>
+  <gazebo reference="${name}_finger_right">
+    <material>Gazebo/White</material>
+    <turnGravityOff>false</turnGravityOff>
+  </gazebo>
 </xacro:macro>
 </robot>
