Commit message: asd

File: iwtros_descriptions/omronld/omronld_description/urdf/omronld.urdf.xacro (robot description, xacro)
@@ -47,7 +47,4 @@
     <origin xyz="0.2652 0.0 0.201" rpy="${M_PI} 0.0 0.0"/>
   </xacro:sick_lms1xx>
-  <xacro:sick_lms1xx frame="base_laser_fake" parent="base_link" topic="scanBack">
-    <origin xyz="-0.2652 0.0 0.105" rpy="${M_PI} 0.0 ${M_PI}"/>
-  </xacro:sick_lms1xx>
   <!-- GAZEBO PLUGINS--> <!-- http://wiki.ros.org/urdf/Tutorials/Using%20a%20URDF%20in%20Gazebo-->
   <gazebo>

Commit message: new map without the standardzelle

File: iwtros_descriptions/omronld/omronld_description/urdf/omronld.urdf.xacro (robot description, xacro)
@@ -44,6 +44,9 @@
   </xacro:omronld_wheel>
   <!-- LASER -->
-  <xacro:sick_lms1xx frame="base_laser" parent="base_link" topic="scan">
+  <xacro:sick_lms1xx frame="base_laser" parent="base_link" topic="scanFront">
     <origin xyz="0.2652 0.0 0.201" rpy="${M_PI} 0.0 0.0"/>
+  </xacro:sick_lms1xx>
+  <xacro:sick_lms1xx frame="base_fake_laser" parent="base_link" topic="scanBack">
+    <origin xyz="-0.2652 0.0 0.105" rpy="${M_PI} 0.0 ${M_PI}"/>
   </xacro:sick_lms1xx>
   <!-- GAZEBO PLUGINS--> <!-- http://wiki.ros.org/urdf/Tutorials/Using%20a%20URDF%20in%20Gazebo-->

Commit message: 3D camera on omron

File: iwtros_descriptions/omronld/omronld_description/urdf/omronld.urdf.xacro (robot description, xacro)
@@ -17,4 +17,5 @@
   <!-- LASER -->
   <xacro:include filename="$(find omronld_description)/urdf/laser/sick_lms1xx.urdf.xacro" />
+  <xacro:include filename="$(find robots_ee_pkg)/urdf/camera/r200.urdf.xacro"/>
   <!-- base_link origin point is center of rotation, on the floor. -->
   <link name="base_link">
@@ -50,4 +51,7 @@
     <origin xyz="-0.2652 0.0 0.105" rpy="${M_PI} 0.0 ${M_PI}"/>
   </xacro:sick_lms1xx>
+  <xacro:camera_r200 parent="base_link">
+        <origin xyz="0.3 0 0.38" rpy="0 0 0" />
+    </xacro:camera_r200>
   <!-- GAZEBO PLUGINS--> <!-- http://wiki.ros.org/urdf/Tutorials/Using%20a%20URDF%20in%20Gazebo-->
   <gazebo>

File: iwtros_descriptions/robots_ee_pkg/urdf/camera/r200.urdf.xacro (robot description, xacro)
@@ -27,10 +27,10 @@
             <!-- This inertial field needs doesn't contain reliable data!! -->
             <inertial>
-            <mass value="0.564" />
+                <mass value="0.564" />
                 <origin xyz="0 0 0" />
-                <inertia ixx="0.003881243" ixy="0.0" ixz="0.0"
-                        iyy="0.000498940" iyz="0.0"
-                        izz="0.003879257" />
-            </inertial>>
+                    <inertia ixx="0.003881243" ixy="0.0" ixz="0.0"
+                            iyy="0.000498940" iyz="0.0"
+                            izz="0.003879257" />
+            </inertial>
         </link>
         <joint name="camera_rgb_joint" type="fixed">
