Commit message: Implementtion and Test of New Omron URDF
Problem of AMCL is not solved yet

File: iwtros_descriptions/omronld/omronld_description/urdf/new_omronld.urdf.xacro (robot description, xacro)
@@ -2,5 +2,5 @@
 <robot name="omronld" xmlns:xacro="http://ros.org/wiki/xacro">
   <!--general-->
-  <xacro:arg name="robot_description" default="robot_description" />
+  <xacro:arg name="robot_description" default="omronld_description" />
   <xacro:property name="M_PI" value="3.14159"/>
   <!--wheels-->
@@ -17,4 +17,5 @@
   <!-- LASER -->
   <xacro:include filename="$(find omronld_description)/urdf/laser/sick_lms1xx.urdf.xacro" />
+  <xacro:include filename="$(find robots_ee_pkg)/urdf/camera/r200.urdf.xacro"/>
   <!-- base_link origin point is center of rotation, on the floor. -->
   <link name="base_link">
@@ -31,5 +32,5 @@
     <collision name="base_link_collision">
       <geometry name="base_link_collision_geom">
-        <box size="0.7 0.5 0.05" />
+        <box size="0.7 0.5 0.001" />
       </geometry>
       <origin xyz="0 0 0.1" rpy="0 0 0" />
@@ -37,12 +38,12 @@
   </link>
   <!-- omronld wheel macros -->
-  <xacro:omronld_wheel wheel_prefix="l_wheel">
+  <xacro:omronld_wheel wheel_prefix="left">
     <origin xyz="${wheelbase/2} ${track/2} ${wheel_vertical_offset}" rpy="0 0 0" />
   </xacro:omronld_wheel>
-  <xacro:omronld_wheel wheel_prefix="r_wheel">
+  <xacro:omronld_wheel wheel_prefix="right">
     <origin xyz="${wheelbase/2} ${-track/2} ${wheel_vertical_offset}" rpy="0 0 0" />
   </xacro:omronld_wheel>
   <!-- LASER -->
-  <xacro:sick_lms1xx frame="base_laser" parent="base_link" topic="scanFront">
+  <xacro:sick_lms1xx frame="base_laser" parent="base_link" topic="scanFront" >
     <origin xyz="0.2652 0.0 0.201" rpy="${M_PI} 0.0 0.0"/>
   </xacro:sick_lms1xx>
@@ -50,8 +51,12 @@
     <origin xyz="-0.2652 0.0 0.105" rpy="${M_PI} 0.0 ${M_PI}"/>
   </xacro:sick_lms1xx>
+  <!--xacro:camera_r200 parent="base_link">
+        <origin xyz="0.3 0 0.38" rpy="0 0 0" />
+    </xacro:camera_r200-->
   <!-- GAZEBO PLUGINS--> <!-- http://wiki.ros.org/urdf/Tutorials/Using%20a%20URDF%20in%20Gazebo-->
   <gazebo>
     <plugin name="gazebo_ros_control" filename="libgazebo_ros_control.so">
-      <robotNamespace>$(arg robot_description)</robotNamespace>
+      <legacyModeNS>false</legacyModeNS>
+      <robotNamespace>$(arg robot_namespace)</robotNamespace>
     </plugin>
   </gazebo>
