Commit message: Redefine URDF and update MovieIt for Joint State: PTP is successful
Checking the robot kinematic before the MotionPlanningReq message is set using "void moveit::planning_interface::MoveGroupInterface setTrajectoryConstraints(moveit_msgs::TrajectoryConstraints& contraints) is important.

File: iiwa_stack-master/iiwa_description/urdf/iiwa7.xacro (robot description, xacro)
@@ -54,5 +54,5 @@
       <axis xyz="0 0 1"/>
       <limit lower="${-170 * PI / 180}" upper="${170 * PI / 180}"
-             effort="${max_effort}" velocity="${max_velocity}" />
+             effort="${max_effort}" velocity="${98 * PI / 180}" />
       <safety_controller soft_lower_limit="${-168 * PI / 180}"
                          soft_upper_limit="${168 * PI / 180}"
@@ -88,5 +88,5 @@
       <axis xyz="0 0 1"/>
       <limit lower="${-120 * PI / 180}" upper="${120 * PI / 180}"
-             effort="${max_effort}" velocity="${max_velocity}" />
+             effort="${max_effort}" velocity="${98 * PI / 180}" />
       <safety_controller soft_lower_limit="${-118 * PI / 180}"
                          soft_upper_limit="${118 * PI / 180}"
@@ -122,5 +122,5 @@
       <axis xyz="0 0 1"/>
       <limit lower="${-170 * PI / 180}" upper="${170 * PI / 180}"
-             effort="${max_effort}" velocity="${max_velocity}" />
+             effort="${max_effort}" velocity="${100 * PI / 180}" />
       <safety_controller soft_lower_limit="${-168 * PI / 180}"
                          soft_upper_limit="${168 * PI / 180}"
@@ -156,5 +156,5 @@
       <axis xyz="0 0 1"/>
       <limit lower="${-120 * PI / 180}" upper="${120 * PI / 180}"
-             effort="${max_effort}" velocity="${max_velocity}" />
+             effort="${max_effort}" velocity="${130 * PI / 180}" />
       <safety_controller soft_lower_limit="${-118 * PI / 180}"
                          soft_upper_limit="${118 * PI / 180}"
@@ -190,5 +190,5 @@
       <axis xyz="0 0 1"/>
       <limit lower="${-170 * PI / 180}" upper="${170 * PI / 180}"
-             effort="${max_effort}" velocity="${max_velocity}" />
+             effort="${max_effort}" velocity="${140 * PI / 180}" />
       <safety_controller soft_lower_limit="${-168 * PI / 180}"
                          soft_upper_limit="${168 * PI / 180}"
@@ -224,5 +224,5 @@
       <axis xyz="0 0 1"/>
       <limit lower="${-120 * PI / 180}" upper="${120 * PI / 180}"
-             effort="${max_effort}" velocity="${max_velocity}" />
+             effort="${max_effort}" velocity="${180 * PI / 180}" />
       <safety_controller soft_lower_limit="${-118 * PI / 180}"
                          soft_upper_limit="${118 * PI / 180}"
@@ -258,5 +258,5 @@
       <axis xyz="0 0 1"/>
       <limit lower="${-175 * PI / 180}" upper="${175 * PI / 180}"
-             effort="${max_effort}" velocity="${max_velocity}" />
+             effort="${max_effort}" velocity="${180 * PI / 180}" />
       <safety_controller soft_lower_limit="${-173 * PI / 180}"
                          soft_upper_limit="${173 * PI / 180}"

File: iiwa_stack-master/iiwa_description/urdf/kuka_iiwa7.xacro (robot description, xacro)
@@ -52,5 +52,5 @@
       <axis xyz="0 0 1"/>
       <limit lower="${-170 * PI / 180}" upper="${170 * PI / 180}"
-             effort="${max_effort}" velocity="${max_velocity}" />
+             effort="${max_effort}" velocity="${98 * PI / 180}" />
       <safety_controller soft_lower_limit="${-168 * PI / 180}"
                          soft_upper_limit="${168 * PI / 180}"
@@ -86,5 +86,5 @@
       <axis xyz="0 0 1"/>
       <limit lower="${-120 * PI / 180}" upper="${120 * PI / 180}"
-             effort="${max_effort}" velocity="${max_velocity}" />
+             effort="${max_effort}" velocity="${98 * PI / 180}" />
       <safety_controller soft_lower_limit="${-118 * PI / 180}"
                          soft_upper_limit="${118 * PI / 180}"
@@ -120,5 +120,5 @@
       <axis xyz="0 0 1"/>
       <limit lower="${-170 * PI / 180}" upper="${170 * PI / 180}"
-             effort="${max_effort}" velocity="${max_velocity}" />
+             effort="${max_effort}" velocity="${100 * PI / 180}" />
       <safety_controller soft_lower_limit="${-168 * PI / 180}"
                          soft_upper_limit="${168 * PI / 180}"
@@ -154,5 +154,5 @@
       <axis xyz="0 0 1"/>
       <limit lower="${-120 * PI / 180}" upper="${120 * PI / 180}"
-             effort="${max_effort}" velocity="${max_velocity}" />
+             effort="${max_effort}" velocity="${130 * PI / 180}" />
       <safety_controller soft_lower_limit="${-118 * PI / 180}"
                          soft_upper_limit="${118 * PI / 180}"
@@ -188,5 +188,5 @@
       <axis xyz="0 0 1"/>
       <limit lower="${-170 * PI / 180}" upper="${170 * PI / 180}"
-             effort="${max_effort}" velocity="${max_velocity}" />
+             effort="${max_effort}" velocity="${140 * PI / 180}" />
       <safety_controller soft_lower_limit="${-168 * PI / 180}"
                          soft_upper_limit="${168 * PI / 180}"
@@ -222,5 +222,5 @@
       <axis xyz="0 0 1"/>
       <limit lower="${-120 * PI / 180}" upper="${120 * PI / 180}"
-             effort="${max_effort}" velocity="${max_velocity}" />
+             effort="${max_effort}" velocity="${180 * PI / 180}" />
       <safety_controller soft_lower_limit="${-118 * PI / 180}"
                          soft_upper_limit="${118 * PI / 180}"
@@ -256,5 +256,5 @@
       <axis xyz="0 0 1"/>
       <limit lower="${-175 * PI / 180}" upper="${175 * PI / 180}"
-             effort="${max_effort}" velocity="${max_velocity}" />
+             effort="${max_effort}" velocity="${180 * PI / 180}" />
       <safety_controller soft_lower_limit="${-173 * PI / 180}"
                          soft_upper_limit="${173 * PI / 180}"

File: iwtros_descriptions/robots_ee_pkg/urdf/kuka_robot/kuka_iiwa7_system.urdf (robot description, URDF)
Before this commit: robot kuka_iiwa7_system, 18 links, 17 joints
Joints:
- joint iiwa_joint_1: limit lower=-2.96705972839 upper=2.96705972839 effort=300 velocity=10 -> lower=-2.96705972839 upper=2.96705972839 effort=300 velocity=1.71042266695
- joint iiwa_joint_2: limit lower=-2.09439510239 upper=2.09439510239 effort=300 velocity=10 -> lower=-2.09439510239 upper=2.09439510239 effort=300 velocity=1.71042266695
- joint iiwa_joint_3: limit lower=-2.96705972839 upper=2.96705972839 effort=300 velocity=10 -> lower=-2.96705972839 upper=2.96705972839 effort=300 velocity=1.74532925199
- joint iiwa_joint_4: limit lower=-2.09439510239 upper=2.09439510239 effort=300 velocity=10 -> lower=-2.09439510239 upper=2.09439510239 effort=300 velocity=2.26892802759
- joint iiwa_joint_5: limit lower=-2.96705972839 upper=2.96705972839 effort=300 velocity=10 -> lower=-2.96705972839 upper=2.96705972839 effort=300 velocity=2.44346095279
- joint iiwa_joint_6: limit lower=-2.09439510239 upper=2.09439510239 effort=300 velocity=10 -> lower=-2.09439510239 upper=2.09439510239 effort=300 velocity=3.14159265359
- joint iiwa_joint_7: limit lower=-3.05432619099 upper=3.05432619099 effort=300 velocity=10 -> lower=-3.05432619099 upper=3.05432619099 effort=300 velocity=3.14159265359
- joint wsg50_guide_joint_finger_left: origin xyz=0 0 0.023 rpy=0 0 0 -> xyz=-0.001 0 0.023 rpy=0 0 0
- joint wsg50_guide_joint_finger_right: origin xyz=0 0 0.023 rpy=0 0 0 -> xyz=-0.001 0 0.023 rpy=0 0 0
